File: nightshade.kicad_pcb (KiCad board)
At the start: 4 copper layers, 154.9 x 75.5 mm, 98 parts, among them J1 Conn_02x13_Odd_Even, J2 Bus_ISA_16bit, J3 DB15_Female_HighDensity_Mount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, U1 GD542x_ISA, U2 SOJ_256Kx16, U3 SOJ_256Kx16, U4 LM334SM, U5 27C010, U6 'LS/ALS/F244, U7 SOJ_256Kx16, U8 SOJ_256Kx16, Y1 14.31818MHz

Commit message: Add files via upload
Parts:
- moved C30 15.3 mm to (134.0, 127.2)
Other:
- board text added: "ISA Version 0.8b1 Designed by AB"
- board text removed: "ISA Version 0.8b Designed by AB"

Commit message: Add files via upload
Updated to 0.8b2
Parts:
- U4: value LM334SM -> LM334M
- moved D1 6.04 mm to (195.5, 91.5), turned to -90 degrees
- moved R14 1.58 mm to (193.5, 91.0)
- moved U4 0.64 mm to (202.5, 92.7)
- moved R15 0.56 mm to (197.5, 91.8), turned to -90 degrees
Connections:
- U4 pad 1: Net-(D1-A) -> Net-(R14-Pad2)
- U4 pad 2: Net-(R14-Pad2) -> Net-(D1-A)
- U4 pad 3: /IREF -> Net-(D1-A)
- U4 pad 4: (no net) -> /IREF
- U4 pad 6: (no net) -> Net-(D1-A)
- U4 pad 7: (no net) -> Net-(D1-A)
Routing:
- net Net-(D1-A): track 4.89 -> 22.2 mm
- net Net-(R14-Pad2): track 5.47 -> 6.99 mm
Other:
- board text added: "ISA Version 0.8b2 Designed by AB"
- board text removed: "ISA Version 0.8b1 Designed by AB"

Commit message: Add files via upload
Updated to version 0.8c.
Parts:
- added C9: 0.22u, Capacitor_SMD:C_0805_2012Metric, B.Cu at (219.4, 140.2)
- added U9: LF50_TO252, Package_TO_SOT_SMD:TO-252-2, B.Cu at (228.0, 137.0)
- C12, C13: value C_Small -> 15p
- C16, C27, R12, R19, R22: moved to B.Cu
- C31: value 0.22u -> 22u; footprint Capacitor_SMD:C_0805_2012Metric -> Capacitor_SMD:C_Elec_4x5.8; moved to B.Cu
- C7, C8: value 0.1u -> 10u; footprint Capacitor_SMD:C_0805_2012Metric -> Capacitor_SMD:C_1206_3216Metric
- moved R18 35.5 mm to (176.8, 102.4)
- moved R17 35.5 mm to (176.8, 105.8)
- moved R16 35.5 mm to (176.8, 109.2)
- moved C31 12.6 mm to (225.5, 128.5)
- moved JP3 9.34 mm to (203.9, 138.8)
- moved R22 8.58 mm to (223.9, 132.0), turned to 0 degrees
- moved R19 5.91 mm to (188.9, 131.8)
- moved C18 4.50 mm to (174.1, 142.5), turned to 180 degrees
- moved R12 3.70 mm to (175.6, 143.5), turned to 180 degrees
- moved C16 3.64 mm to (172.8, 144.5), turned to 90 degrees
- moved R13 2.46 mm to (182.2, 141.0), turned to 180 degrees
- moved C7 2.36 mm to (170.9, 109.8), turned to 90 degrees
- moved C8 2.36 mm to (162.0, 98.5), turned to 0 degrees
- moved R8 2.30 mm to (132.0, 114.8)
- moved C27 2.26 mm to (186.2, 132.6), turned to 90 degrees
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Connections:
- J2 pad 9: /+12V -> +12V
- U6 pad 12: /SD4 -> /SD7
- U6 pad 14: /SD5 -> /SD6
- U6 pad 16: /SD6 -> /SD5
- U6 pad 18: /SD7 -> /SD4
- U6 pad 2: /BD7 -> /BD4
- U6 pad 4: /BD6 -> /BD5
- U6 pad 6: /BD5 -> /BD6
- U6 pad 8: /BD4 -> /BD7
Routing:
- net +12V: track 0.00 -> 37.2 mm
- net GND: track 179.7 -> 159.6 mm, vias 156 -> 213
- net /AVcc: track 103.9 -> 88.0 mm, vias 2 -> 1
- net /MID1: track 30.9 -> 21.6 mm
- net /VCC: track 168.0 -> 159.2 mm
- net /BD4: track 19.7 -> 28.3 mm
- net /MID0: track 28.0 -> 19.4 mm, vias 0 -> 2
- net /BD7: track 31.1 -> 22.7 mm
- net /ROM_ENA: track 66.4 -> 73.4 mm
- net Net-(J2-~{SMEMR}): track 23.1 -> 17.7 mm, vias 1 -> 0
- net Net-(U1-RAS): track 3.29 -> 8.00 mm, vias 0 -> 2
- net /BD6: track 28.1 -> 23.5 mm
- net /SA15: track 29.7 -> 25.7 mm
- net /CAS0: track 19.8 -> 15.9 mm
- net /VSYNC: track 90.8 -> 87.0 mm
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Other:
- board text added: "DANGER: Do Not Lick!"
- board text added: "ISA Version 0.8c Designed by AB"
- board text added: "Licking a live linear regulator is generally not a great idea unless you like to smell your hand after pumping gasoline."
- board text added: "Only install R22 if not installing regulator at U9!"
- board text added: "This is *NOT* a Wave Blaster header"
- board text removed: "ISA Version 0.8b2 Designed by AB"
- board text removed: "This is *NOT* a floppy connector"

Commit message: Add files via upload
updated to 0.8c1.
Parts:
- U5: footprint Package_LCC:PLCC-32_11.4x14.0mm_P1.27mm -> SOJ_DRAM:PLCC-32_SMD-Socket
- moved C41 3.54 mm to (221.7, 114.5), turned to 180 degrees
- moved JP2 1.46 mm to (217.2, 112.5), turned to -90 degrees
- moved R24 1.03 mm to (211.2, 114.8)
- moved R25 0.71 mm to (216.8, 114.8)
- moved JP1 0.59 mm to (213.2, 112.5), turned to -90 degrees
- moved U5 0.56 mm to (214.8, 126.5)
- moved JP3 0.50 mm to (203.9, 139.2)
Routing:
- net /VCC: track 159.2 -> 162.2 mm
- net /A16: track 6.37 -> 8.71 mm
- net /A15: track 5.73 -> 7.59 mm
- net /BD0: track 16.0 -> 17.8 mm
- net /SA12: track 76.9 -> 78.0 mm
- net /SA9: track 91.6 -> 90.5 mm
- net /SA2: track 86.9 -> 87.8 mm
- net /SA8: track 93.0 -> 92.0 mm
- net /SA1: track 92.8 -> 93.6 mm
- net /SA0: track 98.1 -> 98.9 mm
- net /SA7: track 80.7 -> 81.4 mm
- net /SA4: track 89.4 -> 90.0 mm
- net /SA11: track 90.2 -> 89.6 mm
- net /IRQ2: track 14.7 -> 14.2 mm
- net GND: vias 213 -> 210
Other:
- board text added: "ISA Version 0.8c1 Designed by AB"
- board text removed: "ISA Version 0.8c Designed by AB"

Commit message: Add files via upload
Updated to Version 0.8c2.
Parts:
- C31, C9, R22, U9: moved to F.Cu
- moved R22 12.4 mm to (235.0, 137.4), turned to -90 degrees
- moved C31 11.9 mm to (231.5, 138.8), turned to -90 degrees
- moved U9 8.26 mm to (229.2, 128.8), turned to 90 degrees
- moved C9 5.60 mm to (225.0, 140.2)
- moved JP1 2.54 mm to (210.7, 112.2), turned to 90 degrees
- moved FID2 0.96 mm to (232.5, 143.6)
- moved JP2 0.63 mm to (217.8, 112.2)
- moved C41 0.51 mm to (221.2, 114.2)
- moved U5 0.46 mm to (214.4, 126.2)
- moved R24 0.20 mm to (211.2, 114.6)
- moved R25 0.20 mm to (216.8, 114.6)
Routing:
- net /AVcc: track 88.0 -> 106.4 mm, vias 1 -> 2
- net +12V: track 37.2 -> 43.8 mm, vias 0 -> 1
- net /SA8: track 92.0 -> 91.2 mm
- net /SA2: track 87.8 -> 87.2 mm
- net /SA14: track 86.2 -> 85.6 mm
- net GND: vias 210 -> 228
Other:
- board text added: "Do not lick LDO Do not kick LDO Usage of LDO to incinerate PCB remains may be a violation of local health ordinances"
- board text added: "ISA Version 0.8c2 Designed by AB"
- board text added: "Only install if not using LDO!"
- board text added: "POSTED:"
- board text removed: "DANGER: Do Not Lick!"
- board text removed: "ISA Version 0.8c1 Designed by AB"
- board text removed: "Licking a live linear regulator is generally not a great idea unless you like to smell your hand after pumping gasoline."
- board text removed: "Only install R22 if not installing regulator at U9!"
